File: 04_Hardware/PCBs/CamTracker/CamTracker.kicad_sch (KiCad schematic)
At the start: 1 part

Commit message: feat: Completed Placement v1 in Layout
Parts:
- removed D1: ~, 000MCLib:DIOM7959X250N, symbol 000MCLib:B520C-13-F
Other:
- note added: "1.05V for NVMe"
- note added: "1.05V/1A"
- note added: "3.3V/3A"
- note added: "3.8V"
- note added: "3V3 for NVMe"
- note added: "SW"
- note removed: "VBAT"
